File: elec/layout/default/drv8300.kicad_pcb (KiCad board)
At the start: 2 copper layers, 225.7 x 100.8 mm, 15 parts

Commit message: added layout
Parts:
- removed R10: Chip Resistor - Surface Mount 39KOhms ±5% 1/16W 0402 RoHS, lib:R0402
- removed R2, R3, R5, R6, R8, R9: Chip Resistor - Surface Mount 10Ohms ±5% 1/16W 0402 RoHS, lib:R0402
- removed R4, R7: Chip Resistor - Surface Mount 4.7KOhms ±5% 1/16W 0402 RoHS, lib:R0402
- C1, C2, C3, C4: value 25V 1uF X5R ±10% 0402 Multilayer Ceramic Capacitors MLCC - SMD/SMT ROHS -> 50V 1uF X5R ±10% 0603 Multilayer Ceramic Capacitors MLCC - SMD/SMT ROHS; footprint lib:C0402 -> lib:C0603
- R1: value Chip Resistor - Surface Mount 4.7KOhms ±5% 1/16W 0402 RoHS -> 62.5mW Thick Film Resistors ±100ppm/℃ ±1% 40.2kΩ 0402 Chip Resistor - Surface Mount ROHS
- moved C1 90.6 mm to (239.0, 98.2), turned to -90 degrees
- moved R1 90.4 mm to (239.0, 95.4), turned to 180 degrees
- moved C2 89.7 mm to (244.8, 93.2), turned to 0 degrees
- moved U1 87.9 mm to (242.5, 96.5)
- moved C4 87.7 mm to (244.8, 99.8), turned to 180 degrees
- moved C3 87.2 mm to (246.2, 96.6), turned to -90 degrees
Connections:
- C1 pad 1: vcc-27 -> vcc
- C1 pad 2: gnd-10 -> gnd
- C2 pad 1: vcc-7 -> ic-vcc
- C2 pad 2: gnd-9 -> vcc-14
- C3 pad 1: vcc-14 -> ic-vcc-1
- C3 pad 2: gnd-9 -> vcc-15
- C4 pad 1: vcc-21 -> ic-vcc-2
- C4 pad 2: gnd-9 -> vcc-16
- R1 pad 1: vcc-10 -> vcc-3
- U1 pad 1: vcc-6 -> vcc-2
- U1 pad 10: vcc-16 -> vcc-9
- U1 pad 11: vcc-9 -> vcc-8
- U1 pad 12: vcc-21 -> vcc-16
- U1 pad 13: vcc-22 -> vcc-13
- U1 pad 14: vcc-26 -> ic-vcc-2
- U1 pad 15: vcc-14 -> vcc-15
- U1 pad 16: vcc-15 -> vcc-12
- U1 pad 17: vcc-25 -> ic-vcc-1
- U1 pad 18: vcc-7 -> vcc-14
- U1 pad 19: vcc-8 -> vcc-11
- U1 pad 2: vcc-13 -> vcc-3
- U1 pad 20: gnd-9 -> ic-vcc
- U1 pad 22: vcc-6 -> vcc-5
- U1 pad 23: vcc-13 -> vcc-6
- U1 pad 24: vcc-20 -> vcc-7
- U1 pad 3: vcc-20 -> vcc-4
- U1 pad 4: vcc-1 -> vcc
- U1 pad 5: vcc-1 -> vcc-17
- U1 pad 9: vcc-23 -> vcc-10
Routing:
- net gnd: track 0.00 -> 8.87 mm
- net ic-vcc-2: track 0.00 -> 3.32 mm
- net vcc-14: track 0.00 -> 2.61 mm
- net vcc-15: track 0.00 -> 2.04 mm
- net ic-vcc-1: track 0.00 -> 1.81 mm
- net ic-vcc: track 0.00 -> 1.77 mm
- net vcc-16: track 0.00 -> 1.46 mm
- net vcc-3: track 0.00 -> 1.26 mm

Commit message: minor layout fix
Routing:
- net vcc: track 0.00 -> 1.86 mm
Changed lines of the file:
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@@
   (segment (start 238.2 95.4) (end 238 95.6) (width 0.25) (layer "F.Cu") (net 5))
   (segment (start 238.49 95.4) (end 238.2 95.4) (width 0.25) (layer "F.Cu") (net 5))
-  (segment (start 239.425 98.975) (end 240.6 97.8) (width 0.25) (layer "F.Cu") (net 5))
   (segment (start 238 97.975) (end 239 98.975) (width 0.25) (layer "F.Cu") (net 5))
+  (segment (start 239.025 98.975) (end 240.2 97.8) (width 0.25) (layer "F.Cu") (net 5))
   (segment (start 240.6 97.8) (end 241.25 97.8) (width 0.25) (layer "F.Cu") (net 5))
-  (segment (start 239 98.975) (end 239.425 98.975) (width 0.25) (layer "F.Cu") (net 5))
+  (segment (start 240.2 97.8) (end 240.6 97.8) (width 0.25) (layer "F.Cu") (net 5))
+  (segment (start 239 98.975) (end 239.025 98.975) (width 0.25) (layer "F.Cu") (net 5))
   (segment (start 243.75 98.45) (end 243.75 99.525) (width 0.25) (layer "F.Cu") (net 6))
   (segment (start 243.75 99.525) (end 244.025 99.8) (width 0.25) (layer "F.Cu") (net 6))
@@
   (segment (start 244.425 95.825) (end 244.4 95.8) (width 0.25) (layer "F.Cu") (net 19))
   (segment (start 246.2 95.825) (end 244.425 95.825) (width 0.25) (layer "F.Cu") (net 19))
+  (segment (start 239 97.425) (end 239.625 96.8) (width 0.25) (layer "F.Cu") (net 21))
+  (segment (start 239.625 96.8) (end 240.6 96.8) (width 0.25) (layer "F.Cu") (net 21))
   (group "" (id 6c1ef9f7-0f34-47bb-ac1a-76df23fb396e)
     (members

Commit message: added a lot of layout
Parts:
- moved C3 1.30 mm to (247.5, 96.3)
- moved R1 1.04 mm to (238.0, 95.7), turned to -90 degrees
- moved C1 1.00 mm to (238.0, 98.2)
- moved C2 0.40 mm to (245.2, 93.2)
- moved C4 0.20 mm to (245.0, 99.8)
Routing:
- net vcc-10: track 0.00 -> 2.56 mm, vias 0 -> 1
- net vcc-9: track 0.00 -> 1.94 mm, vias 0 -> 1
- net vcc-12: track 0.00 -> 1.82 mm, vias 0 -> 1
- net vcc-7: track 0.00 -> 1.60 mm, vias 0 -> 1
- net vcc-3: track 1.26 -> 2.85 mm
- net vcc-11: track 0.00 -> 1.55 mm, vias 0 -> 1
- net vcc-4: track 0.00 -> 1.52 mm, vias 0 -> 1
- net vcc-17: track 0.00 -> 1.52 mm, vias 0 -> 1
- net vcc-13: track 0.00 -> 1.48 mm, vias 0 -> 1
- net vcc-5: track 0.00 -> 1.48 mm, vias 0 -> 1
- net vcc-8: track 0.00 -> 1.45 mm, vias 0 -> 1
- net ic-vcc-1: track 1.81 -> 3.18 mm
- net vcc-6: track 0.00 -> 1.31 mm, vias 0 -> 1
- net vcc-15: track 2.04 -> 3.19 mm
- net vcc: track 1.86 -> 2.86 mm
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
Commit message: added a lot of layout and fix
Routing:
- net vcc-2: track 0.00 -> 1.77 mm
Changed lines of the file:
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@@
   (segment (start 245 97.8) (end 244.4 97.8) (width 0.25) (layer "F.Cu") (net 2))
   (via (at 245.2 98.6) (size 0.8) (drill 0.4) (layers "F.Cu" "B.Cu") (net 2))
+  (segment (start 239.4 94.4) (end 239.2 94.4) (width 0.25) (layer "F.Cu") (net 3))
+  (segment (start 240.6 95.3) (end 240.3 95.3) (width 0.25) (layer "F.Cu") (net 3))
+  (segment (start 240.3 95.3) (end 239.4 94.4) (width 0.25) (layer "F.Cu") (net 3))
   (via (at 239.2 94.4) (size 0.8) (drill 0.4) (layers "F.Cu" "B.Cu") (net 3))
+  (segment (start 240.6 95.8) (end 240.049309 95.8) (width 0.25) (layer "F.Cu") (net 4))
+  (segment (start 240.049309 95.8) (end 239.458202 95.208893) (width 0.25) (layer "F.Cu") (net 4))
   (segment (start 238.004849 95.208893) (end 238 95.204044) (width 0.25) (layer "F.Cu") (net 4))
-  (segment (start 240.2 95.8) (end 239.608893 95.208893) (width 0.25) (layer "F.Cu") (net 4))
-  (segment (start 239.608893 95.208893) (end 238.004849 95.208893) (width 0.25) (layer "F.Cu") (net 4))
-  (segment (start 240.6 95.8) (end 240.2 95.8) (width 0.25) (layer "F.Cu") (net 4))
+  (segment (start 239.458202 95.208893) (end 238.004849 95.208893) (width 0.25) (layer "F.Cu") (net 4))
   (segment (start 237 97.975) (end 238 98.975) (width 0.25) (layer "F.Cu") (net 5))
   (segment (start 240.6 97.8) (end 240.2 97.8) (width 0.25) (layer "F.Cu") (net 5))
